Commit message: se pusieron las inercias encada parte

File: description/robot_core.xacro (robot description, xacro)
@@ -26,4 +26,7 @@
             </geometry>
         </collision>
+        <xacro:inertial_box mass="0.5" x="0.3" y="0.3" z="0.15">
+            <origin xyz="0.15 0 0.075" rpy="0 0 0"/>
+        </xacro:inertial_box>
     </link>
     <!-- left wheel joint -->
@@ -47,4 +50,7 @@
             </geometry>
         </collision>
+        <xacro:inertial_cylinder mass="0.1" length="0.04" radius="0.05">
+            <origin xyz="0 0 0" rpy="0 0 0"/>
+        </xacro:inertial_cylinder>
     </link>
     <!-- right wheel joint -->
@@ -68,4 +74,7 @@
             </geometry>
         </collision>
+        <xacro:inertial_cylinder mass="0.1" length="0.04" radius="0.05">
+            <origin xyz="0 0 0" rpy="0 0 0"/>
+        </xacro:inertial_cylinder>
     </link>
     <!-- caster wheel joint -->
@@ -88,4 +97,7 @@
             </geometry>
         </collision>
+        <xacro:inertial_sphere mass="0.1" radius="0.05">
+            <origin xyz="0 0 0" rpy="0 0 0"/>
+        </xacro:inertial_sphere>
     </link>
 </robot>

Commit message: se puso la descripción de la pieza en el entorno de gazebo

File: description/robot_core.xacro (robot description, xacro)
@@ -29,4 +29,7 @@
             <origin xyz="0.15 0 0.075" rpy="0 0 0"/>
         </xacro:inertial_box>
+        <gazebo reference="chassis">
+        <material>Gazebo/White</material>
+        </gazebo>
     </link>
     <!-- left wheel joint -->
@@ -53,4 +56,7 @@
             <origin xyz="0 0 0" rpy="0 0 0"/>
         </xacro:inertial_cylinder>
+        <gazebo reference="left_wheel">
+        <material>Gazebo/Blue</material>
+        </gazebo>
     </link>
     <!-- right wheel joint -->
@@ -77,4 +83,7 @@
             <origin xyz="0 0 0" rpy="0 0 0"/>
         </xacro:inertial_cylinder>
+        <gazebo reference="right_wheel">
+        <material>Gazebo/Blue</material>
+        </gazebo>
     </link>
     <!-- caster wheel joint -->
@@ -100,4 +109,9 @@
             <origin xyz="0 0 0" rpy="0 0 0"/>
         </xacro:inertial_sphere>
+        <gazebo reference="caster_wheel">
+        <material>Gazebo/Black</material>
+        <mu1 value = "0.001" />
+        <mu2 value = "0.001" />
+        </gazebo>
     </link>
 </robot>
