Commit message: correciones del carro

File: description/gazebo_control.xacro (robot description, xacro)
@@ -10,6 +10,6 @@
             <wheel_diameter>0.1</wheel_diameter>
             <!-- limits -->
-            <max_wheel_torque>200</max_wheel_torque>
-            <max_wheel_acceleration>10.0</max_wheel_acceleration>
+            <max_wheel_torque>100</max_wheel_torque>
+            <max_wheel_acceleration>5.0</max_wheel_acceleration>
             <!-- outputs -->
             <odometry_frame>odom</odometry_frame>

File: description/lidar.xacro (robot description, xacro)
@@ -5,5 +5,5 @@
         <parent link="chassis"/>
         <child link="laser_frame"/>
-        <origin xyz="0.1 0 0.175" rpy="0 0 0"/>
+        <origin xyz="0.15 0 0.175" rpy="0 0 0"/>
     </joint>
     <!-- laser_frame -->

File: description/robot_core.xacro (robot description, xacro)
@@ -106,11 +106,11 @@
             </geometry>
         </collision>
-        <xacro:inertial_sphere mass="0.6" radius="0.05">
+        <xacro:inertial_sphere mass="0.1" radius="0.05">
             <origin xyz="0 0 0" rpy="0 0 0"/>
         </xacro:inertial_sphere>
         <gazebo reference="caster_wheel">
         <material>Gazebo/Black</material>
-        <mu1 value = "0.001" />
-        <mu2 value = "0.001" />
+        <mu1 value = "0.0005" />
+        <mu2 value = "0.0005" />
         </gazebo>
     </link>

Commit message: arreglo de las fisicas del carro

File: description/gazebo_control.xacro (robot description, xacro)
@@ -10,6 +10,6 @@
             <wheel_diameter>0.1</wheel_diameter>
             <!-- limits -->
-            <max_wheel_torque>10</max_wheel_torque>
-            <max_wheel_acceleration>1.0</max_wheel_acceleration>
+            <max_wheel_torque>100</max_wheel_torque>
+            <max_wheel_acceleration>10.0</max_wheel_acceleration>
             <!-- outputs -->
             <odometry_frame>odom</odometry_frame>

File: description/robot_core.xacro (robot description, xacro)
@@ -29,7 +29,4 @@
             <origin xyz="0.15 0 0.075" rpy="0 0 0"/>
         </xacro:inertial_box>
-        <gazebo reference="chassis">
-        <material>Gazebo/White</material>
-        </gazebo>
     </link>
     <!-- left wheel joint -->
@@ -56,7 +53,4 @@
             <origin xyz="0 0 0" rpy="0 0 0"/>
         </xacro:inertial_cylinder>
-        <gazebo reference="left_wheel">
-        <material>Gazebo/Blue</material>
-        </gazebo>
     </link>
     <!-- right wheel joint -->
@@ -83,7 +77,4 @@
             <origin xyz="0 0 0" rpy="0 0 0"/>
         </xacro:inertial_cylinder>
-        <gazebo reference="right_wheel">
-        <material>Gazebo/Blue</material>
-        </gazebo>
     </link>
     <!-- caster wheel joint -->
@@ -106,12 +97,21 @@
             </geometry>
         </collision>
-        <xacro:inertial_sphere mass="0.5" radius="0.05">
+        <xacro:inertial_sphere mass="0.1" radius="0.05">
             <origin xyz="0 0 0" rpy="0 0 0"/>
         </xacro:inertial_sphere>
-        <gazebo reference="caster_wheel">
+    </link>
+    <gazebo reference="chassis">
+        <material>Gazebo/White</material>
+    </gazebo>
+    <gazebo reference="left_wheel">
+        <material>Gazebo/Blue</material>
+    </gazebo>
+    <gazebo reference="right_wheel">
+        <material>Gazebo/Blue</material>
+    </gazebo>
+    <gazebo reference="caster_wheel">
         <material>Gazebo/Black</material>
-        <mu1 value = "2.0" />
-        <mu2 value = "2.0" />
-        </gazebo>
-    </link>
+        <mu1 value = "0.001" />
+        <mu2 value = "0.001" />
+    </gazebo>
 </robot>
